File: hardware/express.kicad_pcb (KiCad board)
At the start: 4 copper layers, 180 x 35 mm, 180 parts, among them J1001 SJ2-25404B-SMT-TR, J101 Cortex, J1101 SJ2-25404B-SMT-TR, J1201 SJ2-25404B-SMT-TR, J1301 SJ2-25404B-SMT-TR, J1401 SJ2-25404B-SMT-TR, J1501 SJ2-25404B-SMT-TR, J1601 SJ2-25404B-SMT-TR, J1701 SJ2-25404B-SMT-TR, J1801 2x05_Horizontal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

Commit message: Update
Parts:
- renumbered C110 to C101, C111 to C102, C101 to C103, C103 to C104, C104 to C105, C105 to C106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
