File: hardware/ExpressionInput.kicad_sch (KiCad schematic)
At the start: 8 parts, among them J201 SJ2-25404B-SMT-TR

Commit message: Replace Order_Number
Parts:
- C201: footprint Capacitor_SMD:C_0603_1608Metric -> V2_Capacitor_SMD:C_0603; symbol Device:C_Small -> V2_Device:C_0603_0u022; Manufacturer (none) -> YAGEO; Mouser (none) -> 603-CC603KPX7R9BB223; Product (none) -> CC0603KPX7R9BB223
- D201: footprint Diode_SMD:D_SOD-523 -> V2_Diode_SMD:D_SOD-523; Manufacturer (none) -> ROHM Semiconductor; Mouser (none) -> 755-RB501SM-30FHT2R; Product (none) -> RB501SM-30FHT2R
- D202: LCSC (none) -> C965555; Manufacturer (none) -> Worldsemi; Product (none) -> WS2812B-2020
- J201: Manufacturer (none) -> Same Sky; Mouser (none) -> 490-SJ2-25404BSMT-TR; Product (none) -> SJ2-25404B-SMT-TR
- R201: footprint Resistor_SMD:R_0603_1608Metric -> V2_Resistor_SMD:R_0603; symbol Device:R_Small -> V2_Device:R_0603_33R; Manufacturer (none) -> Vishay; Mouser (none) -> 71-CRCW060333R0FKEAH; Product (none) -> CRCW060333R0FKEAHP; Rating (none) -> 330mW
- R202: footprint Resistor_SMD:R_0603_1608Metric -> V2_Resistor_SMD:R_0603; symbol Device:R_Small -> V2_Device:R_0603_1k; Manufacturer (none) -> Vishay; Mouser (none) -> 71-CRCW06031K00FKEAH; Product (none) -> CRCW06031K00FKEAHP; Rating (none) -> 330mW
- R203: footprint Resistor_SMD:R_0603_1608Metric -> V2_Resistor_SMD:R_0603; symbol Device:R_Small -> V2_Device:R_0603_100k; Manufacturer (none) -> Vishay; Mouser (none) -> 71-CRCW0603100KFKEAC; Product (none) -> CRCW0603100KFKEAC; Rating (none) -> 100mW
- TVS201: footprint Diode_SMD:D_0603_1608Metric -> V2_Diode_SMD:D_0603; Manufacturer (none) -> Bourns; Mouser (none) -> 652-CG0603MLC-3.3LE; Product (none) -> CG0603MLC-3.3LE; Rating (none) -> 3V3

Commit message: Update Library
Parts:
- C201: symbol V2_Device:C_0603_0u022 -> V2_Capacitor:0603_0u022
- R201: symbol V2_Device:R_0603_33R -> V2_Resistor:0603_33R
- R202: symbol V2_Device:R_0603_1k -> V2_Resistor:0603_1k
- R203: symbol V2_Device:R_0603_100k -> V2_Resistor:0603_100k

Commit message: Replace diode
Parts:
- D201: value RB501SM -> PMEG2010EPK; footprint V2_Diode_SMD:D_SOD-523 -> V2_Diode_SMD:D_SOD-1608; symbol V2_Diode:RB501SM -> V2_Diode:PMEG2010EPK; Manufacturer ROHM Semiconductor -> Nexperia; Mouser 755-RB501SM-30FHT2R -> 771-PMEG2010EPK; Product RB501SM-30FHT2R -> PMEG2010EPK; Rating (none) -> 20V
Other:
- title: Expression Input -> V2 express

Commit message: Update
Parts:
- C201: Id (none) -> Capacitor:${SYMBOL_NAME}; Rating (none) -> 50V
- D201, TVS201: Id (none) -> Diode:${SYMBOL_NAME}
- D202: Id (none) -> LED:${SYMBOL_NAME}
- J201: Id (none) -> Audio:${SYMBOL_NAME}
- R201, R202, R203: Id (none) -> Resistor:${SYMBOL_NAME}
Changed lines of the file:
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@@
+			)
+		)
+		(property "Id" "Resistor:${SYMBOL_NAME}"
+			(at 140.97 67.31 0)
+			(hide yes)
+			(show_name no)
+			(do_not_autoplace no)
+			(effects
+				(font
+					(size 1.27 1.27)
+				)
 			)
 		)
@@
 		(property "Rating" "330mW"
 			(at 132.08 101.6 0)
+			(hide yes)
+			(show_name no)
+			(do_not_autoplace no)
+			(effects
+				(font
+					(size 1.27 1.27)
+				)
+			)
+		)
+		(property "Id" "Resistor:${SYMBOL_NAME}"
+			(at 140.97 101.6 0)
 			(hide yes)
 			(show_name no)
@@
 			)
 		)
+		(property "Id" "Audio:${SYMBOL_NAME}"
+			(at 111.76 119.38 0)
+			(hide yes)
+			(show_name no)
+			(do_not_autoplace no)
+			(effects
+				(font
+					(size 1.27 1.27)
+				)
+			)
+		)
 		(pin "1"
 		)
@@
 		(property "Manufacturer" "YAGEO"
 			(at 198.12 119.38 0)
+			(hide yes)
+			(show_name no)
+			(do_not_autoplace no)
+			(effects
+				(font
+					(size 1.27 1.27)
+				)
+			)
+		)
+		(property "Id" "Capacitor:${SYMBOL_NAME}"
+			(at 198.12 116.84 0)
+			(hide yes)
+			(show_name no)
+			(do_not_autoplace no)
+			(effects
+				(font
+					(size 1.27 1.27)
+				)
+			)
+		)
+		(property "Rating" "50V"
+			(at 198.12 127 0)
 			(hide yes)
 			(show_name no)
@@
 			)
 		)
+		(property "Id" "Diode:${SYMBOL_NAME}"
+			(at 172.72 105.41 0)
+			(hide yes)
+			(show_name no)
+			(do_not_autoplace no)
+			(effects
+				(font
+					(size 1.27 1.27)
+				)
+			)
+		)
 		(pin "1"
 		)
@@
 			)
 		)
+		(property "Id" "Diode:${SYMBOL_NAME}"
+			(at 149.86 86.36 0)
+			(hide yes)
+			(show_name no)
+			(do_not_autoplace no)
+			(effects
+				(font
+					(size 1.27 1.27)
+				)
+			)
+		)
 		(pin "1"
 		)
@@
 			)
 		)
+		(property "Id" "LED:${SYMBOL_NAME}"
+			(at 156.21 147.32 0)
+			(hide yes)
+			(show_name no)
+			(do_not_autoplace no)
+			(effects
+				(font
+					(size 1.27 1.27)
+				)
+			)
+		)
 		(pin "1"
 		)
@@
 			(hide yes)
 			(show_name no)
+			(do_not_autoplace no)
+			(effects
+				(font
+					(size 1.27 1.27)
+				)
+			)
+		)
+		(property "Id" "Resistor:${SYMBOL_NAME}"
+			(at 140.97 118.11 0)
+			(hide yes)
+			(show_name no)

Commit message: Update
Parts:
- D202: Rating (none) -> 15mA
- J201: Rating (none) -> 2.5mm
- renumbered R203 to R202, R202 to R203

Commit message: Good Bye Imperial
Parts:
- C201: footprint V2_Capacitor_SMD:C_0603 -> V2_Capacitor_SMD:C_1608; symbol V2_Capacitor:0603_0u022 -> V2_Capacitor:1608_0u022
- R201: footprint V2_Resistor_SMD:R_0603 -> V2_Resistor_SMD:R_1608; symbol V2_Resistor:0603_33R -> V2_Resistor:1608_33R
- R202: footprint V2_Resistor_SMD:R_0603 -> V2_Resistor_SMD:R_1608; symbol V2_Resistor:0603_100k -> V2_Resistor:1608_100k
- R203: footprint V2_Resistor_SMD:R_0603 -> V2_Resistor_SMD:R_1608; symbol V2_Resistor:0603_1k -> V2_Resistor:1608_1k
Changed lines of the file:
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@@
 	)
 	(symbol
-		(lib_id "V2_Resistor:0603_33R")
+		(lib_id "V2_Resistor:1608_33R")
 		(at 140.97 81.28 180)
 		(unit 1)
@@
 			)
 		)
-		(property "Footprint" "V2_Resistor_SMD:R_0603"
+		(property "Footprint" "V2_Resistor_SMD:R_1608"
 			(at 140.97 65.532 0)
 			(hide yes)
@@
 	)
 	(symbol
-		(lib_id "V2_Resistor:0603_1k")
+		(lib_id "V2_Resistor:1608_1k")
 		(at 154.94 101.6 270)
 		(unit 1)
@@
 			)
 		)
-		(property "Footprint" "V2_Resistor_SMD:R_0603"
+		(property "Footprint" "V2_Resistor_SMD:R_1608"
 			(at 139.192 101.6 0)
 			(hide yes)
@@
 	)
 	(symbol
-		(lib_id "V2_Capacitor:0603_0u022")
+		(lib_id "V2_Capacitor:1608_0u022")
 		(at 198.12 104.14 0)
 		(unit 1)
@@
 			)
 		)
-		(property "Footprint" "V2_Capacitor_SMD:C_0603"
+		(property "Footprint" "V2_Capacitor_SMD:C_1608"
 			(at 198.12 121.158 0)
 			(hide yes)
@@
 	)
 	(symbol
-		(lib_id "V2_Resistor:0603_100k")
+		(lib_id "V2_Resistor:1608_100k")
 		(at 140.97 104.14 0)
 		(unit 1)
@@
 			)
 		)
-		(property "Footprint" "V2_Resistor_SMD:R_0603"
+		(property "Footprint" "V2_Resistor_SMD:R_1608"
 			(at 140.97 119.888 0)
 			(hide yes)
