File: hardware/express.kicad_sch (KiCad schematic)
At the start: 44 parts, among them J101 Cortex_Debug, SW101 SW_Push, SW102 SW_Push, U101 TPS78433QWDRBRQ1, U102 ATSAMD51J, Y101 32k768

Commit message: Replace Order_Number
Parts:
- C101: footprint Capacitor_SMD:C_0603_1608Metric -> V2_Capacitor_SMD:C_0603; symbol Device:C_Small -> V2_Device:C_0603_10u; Manufacturer (none) -> TDK; Mouser (none) -> 810-C1608X6S1A106M; Product (none) -> C1608X6S1A106M080AC; Rating (none) -> 10V
- C103, C104, C105, C106, C107: footprint Capacitor_SMD:C_0603_1608Metric -> V2_Capacitor_SMD:C_0603; symbol Device:C_Small -> V2_Device:C_0603_0u1; Manufacturer (none) -> TDK; Mouser (none) -> 810-CGA3E2X7R1H104MA; Product (none) -> CGA3E2X7R1H104M080AA; Rating (none) -> 50V
- C108, C109: footprint Capacitor_SMD:C_0603_1608Metric -> V2_Capacitor_SMD:C_0805; symbol Device:C_Small -> V2_Device:C_0805_10u; Manufacturer (none) -> TDK; Mouser (none) -> 810-C2012X5R1E106K; Product (none) -> C2012X5R1E106K125AB; Rating (none) -> 25V
- C110, C111: footprint Capacitor_SMD:C_0603_1608Metric -> V2_Capacitor_SMD:C_0603; symbol Device:C_Small -> V2_Device:C_0603_18p; Manufacturer (none) -> YAGEO; Mouser (none) -> 603-CC603JRNPO9BN180; Product (none) -> CC0603JRNPO9BN180
- D101, D102: LCSC (none) -> C965555; Manufacturer (none) -> Worldsemi; Product (none) -> WS2812B-2020
- D103: footprint LED_SMD:LED_0603_1608Metric -> V2_LED:LED_0603; symbol Device:LED_Small -> V2_Device:LED_0603_Orange; Manufacturer (none) -> ROHM Semiconductor; Mouser (none) -> 755-SML-D12D1WT86; Product (none) -> SML-D12D1WT86
- ESD101: Manufacturer (none) -> Semtech; Mouser (none) -> 947-RCLAMP0582N.TCT; Product (none) -> RCLAMP0582N.TCT
- FID101, FID102, FID103: value Fiducial -> Fiducial_Paste
- H101, H102, H105: value MountingHole_3mm -> 3mm
- H103, H104, H106, H107, H108: value MountingHole_2mm -> 2mm
- INFO101: value Order_Number -> (none); footprint V2_Production:Order_Number -> V2_Production:Revision; symbol V2_Production:Order_Number -> V2_Production:Revision
- J101: value Cortex_Debug -> Cortex; footprint V2_Cortex_Debug:Cortex_Debug_Pad -> V2_Connector_Debug:Cortex; symbol V2_Cortex_Debug:Cortex_Debug -> V2_Connector_Debug:Cortex
- R101: footprint Resistor_SMD:R_0603_1608Metric -> V2_Resistor_SMD:R_0603; symbol Device:R_Small -> V2_Device:R_0603_330R; Manufacturer (none) -> Vishay; Mouser (none) -> 71-CRCW0603330RFKEAC; Product (none) -> CRCW0603330RFKEAC; Rating (none) -> 100mW
- R102: footprint Resistor_SMD:R_0603_1608Metric -> V2_Resistor_SMD:R_0603; symbol Device:R_Small -> V2_Device:R_0603_100k; Manufacturer (none) -> Vishay; Mouser (none) -> 71-CRCW0603100KFKEAC; Product (none) -> CRCW0603100KFKEAC; Rating (none) -> 100mW
- SW101, SW102: value SW_Push -> SKSG; symbol Switch:SW_Push -> V2_Switch:SKSG; Manufacturer (none) -> Alps Alpine; Mouser (none) -> 688-SKSGACE010; Product (none) -> SKSGACE010
- TVS101: footprint Diode_SMD:D_0603_1608Metric -> V2_Diode_SMD:D_0603; Manufacturer (none) -> Bourns; Mouser (none) -> 652-CG0603MLC-05LE; Product (none) -> CG0603MLC-05LE; Rating (none) -> 5V
- TVS102: footprint Diode_SMD:D_0603_1608Metric -> V2_Diode_SMD:D_0603; Manufacturer (none) -> Bourns; Mouser (none) -> 652-CG0603MLC-3.3LE; Product (none) -> CG0603MLC-3.3LE; Rating (none) -> 3V3
- U101: Manufacturer (none) -> Texas Instruments; Mouser (none) -> 595-TPS78433QWDRBRQ1; Product (none) -> TPS78433QWDRBRQ1
- U102: Manufacturer (none) -> Microchip Technology; Mouser (none) -> 556-ATSAMD51J19AMU; Product (none) -> ATSAMD51J19A-MU
- Y101: symbol Device:Crystal_Small -> V2_Device:Crystal_3.2x1.5_32k768; Manufacturer (none) -> ABRACON; Mouser (none) -> 815-ABS0716632.768KT; Product (none) -> ABS07-166-32.768KHZ-T
Other:
- moved on the sheet: FID101, FID102, FID103, H101, H102, H103, H104, H105, H106, H107, H108, ICON101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

Commit message: Update Library
Parts:
- C101: symbol V2_Device:C_0603_10u -> V2_Capacitor:0603_10u
- C103, C104, C105, C106, C107: symbol V2_Device:C_0603_0u1 -> V2_Capacitor:0603_0u1
- C108, C109: symbol V2_Device:C_0805_10u -> V2_Capacitor:0805_10u
- C110, C111: symbol V2_Device:C_0603_18p -> V2_Capacitor:0603_18p
- D103: symbol V2_Device:LED_0603_Orange -> V2_LED:0603_Orange
- INFO101: value (none) -> ~
- R101: symbol V2_Device:R_0603_330R -> V2_Resistor:0603_330R
- R102: symbol V2_Device:R_0603_100k -> V2_Resistor:0603_100k
- Y101: symbol V2_Device:Crystal_3.2x1.5_32k768 -> V2_Crystal:3.2x1.5_32k768

Commit message: Update ESD suppressor
Parts:
- C110, C111: Manufacturer YAGEO -> TDK; Mouser 603-CC603JRNPO9BN180 -> 810-CGA3E2C0G1H180J; Product CC0603JRNPO9BN180 -> CGA3E2C0G1H180J080AA
Connections:
- no-connect marks 21 -> 23
Changed lines of the file:
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@@
 	(title_block
 		(title "V2 express")
-		(date "2026-02-10")
+		(date "2026-03-14")
 		(rev "2026-02-10")
 		(company "Versio Duo")
@@
 	)
 	(no_connect
+		(at 196.85 86.36)
+	)
+	(no_connect
+		(at 196.85 78.74)
+	)
+	(no_connect
 		(at 86.36 72.39)
 	)
@@
 	(wire
 		(pts
-			(xy 190.5 81.28) (xy 196.85 81.28)
+			(xy 190.5 83.82) (xy 196.85 83.82)
 		)
 		(stroke
@@
 	(wire
 		(pts
+			(xy 190.5 76.2) (xy 196.85 76.2)
+		)
+		(stroke
+			(width 0)
+			(type default)
+		)
+	)
+	(wire
+		(pts
 			(xy 78.74 154.94) (xy 91.44 154.94)
 		)
@@
 	(wire
 		(pts
-			(xy 190.5 83.82) (xy 196.85 83.82)
-		)
-		(stroke
-			(width 0)
-			(type default)
-		)
-	)
-	(wire
-		(pts
 			(xy 142.24 167.64) (xy 153.67 167.64)
 		)
@@
 		)
 	)
+	(label "USB+"
+		(at 190.5 76.2 0)
+		(effects
+			(font
+				(size 1.27 1.27)
+			)
+			(justify left bottom)
+		)
+	)
 	(label "LED-9"
 		(at 16.51 180.34 0)
@@
 		)
 	)
-	(label "USB+"
-		(at 190.5 83.82 0)
-		(effects
-			(font
-				(size 1.27 1.27)
-			)
-			(justify left bottom)
-		)
-	)
 	(label "Analog-12"
 		(at 153.67 177.8 180)
@@
 	)
 	(label "USB-"
-		(at 190.5 81.28 0)
+		(at 190.5 83.82 0)
 		(effects
 			(font
@@
 		(dnp no)
 		(property "Reference" "ESD101"
-			(at 199.39 73.66 0)
+			(at 199.136 68.834 0)
 			(effects
 				(font
@@
 		)
 		(property "Value" "RCLAMP0582N"
-			(at 199.39 76.835 0)
+			(at 199.136 72.009 0)
 			(effects
 				(font
@@
 			)
 		)
-		(property "Description" "Push button switch, generic, two pins"
+		(property "Description" "Push button"
 			(at 252.73 27.94 0)
 			(effects
@@
 			)
 		)
-		(property "Description" "Unpolarized capacitor, small symbol"
+		(property "Description" ""
 			(at 88.9 35.56 0)
 			(effects
@@
 	(symbol
 		(lib_id "V2_power:+5V")
-		(at 214.63 81.28 270)
+		(at 214.63 76.2 270)
 		(unit 1)
 		(exclude_from_sim no)
@@
 		(fields_autoplaced yes)
 		(property "Reference" "#PWR118"
-			(at 210.82 81.28 0)
+			(at 210.82 76.2 0)
 			(effects
 				(font
@@
 		)
 		(property "Value" "+5V"
-			(at 218.44 81.2799 90)
+			(at 218.44 76.1999 90)
 			(effects
 				(font
@@
 		)
 		(property "Footprint" ""
-			(at 214.63 81.28 0)
+			(at 214.63 76.2 0)
 			(effects
 				(font
@@
 		)
 		(property "Datasheet" ""
-			(at 214.63 81.28 0)
+			(at 214.63 76.2 0)
 			(effects
 				(font
@@
 		)
 		(property "Description" ""
-			(at 214.63 81.28 0)
+			(at 214.63 76.2 0)
 			(effects
 				(font
@@
 			)
 		)
-		(property "Description" "Two pin crystal, small symbol"
+		(property "Description" ""
 			(at 24.13 41.91 0)
 			(effects
@@
 			)
 		)
-		(property "Description" "Light emitting diode, small symbol"
+		(property "Description" ""
 			(at 132.08 55.88 0)
 			(effects
@@
 			)
 		)
-		(property "Description" "Unpolarized capacitor, small symbol"
+		(property "Description" ""
 			(at 201.93 53.34 0)
 			(effects
@@
 			)
 		)
-		(property "Description" "Unpolarized capacitor, small symbol"
+		(property "Description" ""
 			(at 26.67 60.198 0)
 			(effects
@@
 			)
 		)
-		(property "Mouser" "603-CC603JRNPO9BN180"
+		(property "Mouser" "810-CGA3E2C0G1H180J"
 			(at 26.67 69.088 0)
 			(effects
@@
 			)
 		)
-		(property "Product" "CC0603JRNPO9BN180"
+		(property "Product" "CGA3E2C0G1H180J080AA"
 			(at 26.67 66.294 0)
 			(effects
@@
 			)
 		)
-		(property "Manufacturer" "YAGEO"
+		(property "Manufacturer" "TDK"
 			(at 26.67 63.5 0)
 			(effects
@@
 			)
 		)
-		(property "Description" "Unpolarized capacitor, small symbol"
+		(property "Description" ""
 			(at 177.8 53.34 0)
 			(effects
@@
 			)
 		)
-		(property "Description" "Unpolarized capacitor, small symbol"
+		(property "Description" ""
 			(at 119.38 35.56 0)
 			(effects
@@
 			)
 		)
-		(property "Description" "Resistor, small symbol"
+		(property "Description" ""
 			(at 63.5 120.65 0)
 			(effects
@@
 			)
 		)
-		(property "Description" "Unpolarized capacitor, small symbol"
+		(property "Description" ""
 			(at 21.59 60.198 0)
 			(effects
@@
 			)
 		)
-		(property "Mouser" "603-CC603JRNPO9BN180"
+		(property "Mouser" "810-CGA3E2C0G1H180J"
 			(at 21.59 69.088 0)
 			(effects
@@
 			)
 		)
-		(property "Product" "CC0603JRNPO9BN180"
+		(property "Product" "CGA3E2C0G1H180J080AA"
 			(at 21.59 66.294 0)
 			(effects
@@
 			)
 		)
-		(property "Manufacturer" "YAGEO"
+		(property "Manufacturer" "TDK"
 			(at 21.59 63.5 0)
 			(effects
@@
 			)
 		)
-		(property "Description" "Resistor, small symbol"
+		(property "Description" ""
 			(at 152.4 55.88 0)
 			(effects
@@
 	(symbol
 		(lib_id "V2_power:GND")
-		(at 214.63 83.82 90)
+		(at 214.63 86.36 90)
 		(unit 1)
 		(exclude_from_sim no)
@@
 		(fields_autoplaced yes)
 		(property "Reference" "#PWR119"
-			(at 220.98 83.82 0)
+			(at 220.98 86.36 0)
 			(effects
 				(font
@@
 		)
 		(property "Value" "GND"
-			(at 218.44 83.8199 90)
+			(at 218.44 86.3599 90)
 			(effects
 				(font
@@
 		)
 		(property "Footprint" ""
-			(at 214.63 83.82 0)
+			(at 214.63 86.36 0)
 			(effects
 				(font
@@
 		)
 		(property "Datasheet" ""
-			(at 214.63 83.82 0)
+			(at 214.63 86.36 0)
 			(effects
 				(font
@@
 		)
 		(property "Description" ""
-			(at 214.63 83.82 0)
+			(at 214.63 86.36 0)
 			(effects
 				(font
@@
 			)
 		)
-		(property "Description" "Unpolarized capacitor, small symbol"
+		(property "Description" ""
 			(at 99.06 35.56 0)
 			(effects
@@
 			)
 		)
-		(property "Description" "Unpolarized capacitor, small symbol"
+		(property "Description" ""
 			(at 78.74 35.56 0)
 			(effects
@@
 			)
 		)
-		(property "Description" "Push button switch, generic, two pins"
+		(property "Description" "Push button"
 			(at 134.62 73.66 0)
 			(effects
@@
 			)
 		)
-		(property "Description" "Unpolarized capacitor, small symbol"
+		(property "Description" ""
 			(at 109.22 35.56 0)
 			(effects
@@
 			)
 		)
-		(property "Description" "Unpolarized capacitor, small symbol"
+		(property "Description" ""
 			(at 57.15 38.1 0)
 			(effects

Commit message: Replace diode
Parts:
- INFO101: value ~ -> (none)
Other:
- sheet  Expression Input 1 renamed Expression Input 1
- sheet  Expression Input 10 renamed Expression Input 10
- sheet  Expression Input 11 renamed Expression Input 11
- sheet  Expression Input 12 renamed Expression Input 12
- sheet  Expression Input 13 renamed Expression Input 13
- sheet  Expression Input 14 renamed Expression Input 14
- sheet  Expression Input 15 renamed Expression Input 15
- sheet  Expression Input 16 renamed Expression Input 16
- sheet  Expression Input 2 renamed Expression Input 2
- sheet  Expression Input 3 renamed Expression Input 3
- sheet  Expression Input 4 renamed Expression Input 4
- sheet  Expression Input 5  renamed Expression Input 5
- sheet  Expression Input 6 renamed Expression Input 6
- sheet  Expression Input 7 renamed Expression Input 7
- sheet  Expression Input 8 renamed Expression Input 8
- sheet  Expression Input 9 renamed Expression Input 9

Commit message: Update
Parts:
- C101, C103, C104, C105, C106, C107, C108, C109: Id (none) -> Capacitor:${SYMBOL_NAME}
- C110, C111: Id (none) -> Capacitor:${SYMBOL_NAME}; Rating (none) -> 50V
- D101, D102: Id (none) -> LED:${SYMBOL_NAME}
- D103: Id (none) -> LED:${SYMBOL_NAME}; Rating (none) -> 605nm
- ESD101: Id (none) -> ESD:${SYMBOL_NAME}
- R101, R102: Id (none) -> Resistor:${SYMBOL_NAME}
- SW101, SW102: Id (none) -> Button:${SYMBOL_NAME}; Rating (none) -> 1.6N
- TVS101, TVS102: Id (none) -> Diode:${SYMBOL_NAME}
- U101: Id (none) -> LDO:${SYMBOL_NAME}
- U102: Id (none) -> MCU:${SYMBOL_NAME}
- Y101: Id (none) -> Crystal:${SYMBOL_NAME}
Connections:
- net VDDCORE renamed +VDDCORE
Other:
- moved on the sheet: ICON103, INFO101, INFO102

Commit message: Update
Parts:
- D101: renamed from D103; Rating 605nm -> 605nm
- D102: renamed from D101; Rating (none) -> 15mA
- D103: renamed from D102; Rating (none) -> 15mA
- ESD101: Rating (none) -> 20kV
- U101: renamed from U102; Rating (none) -> Cortex-M4F
- U102: renamed from U101; Rating (none) -> 300mA
- Y101: Rating (none) -> 10ppm
- renumbered C110 to C101, C111 to C102, C101 to C103, C103 to C104, C104 to C105, C105 to C106, C106 to C107, C107 to C108, C108 to C109, C109 to C110, H105 to H103, H103 to H104, H104 to H105, ICON103 to ICON101, ICON104 to ICON102, ICON101 to ICON103, ICON102 to ICON104, INFO102 to INFO101, INFO101 to INFO102, R102 to R101, R101 to R102, SW102 to SW101, SW101 to SW102, TVS102 to TVS101, TVS101 to TVS102

Commit message: Good Bye Imperial
Parts:
- C101, C102: footprint V2_Capacitor_SMD:C_0603 -> V2_Capacitor_SMD:C_1608; symbol V2_Capacitor:0603_18p -> V2_Capacitor:1608_18p
- C103: footprint V2_Capacitor_SMD:C_0603 -> V2_Capacitor_SMD:C_1608; symbol V2_Capacitor:0603_10u -> V2_Capacitor:1608_10u
- C104, C105, C106, C107, C108: footprint V2_Capacitor_SMD:C_0603 -> V2_Capacitor_SMD:C_1608; symbol V2_Capacitor:0603_0u1 -> V2_Capacitor:1608_0u1
- C109, C110: footprint V2_Capacitor_SMD:C_0805 -> V2_Capacitor_SMD:C_2012; symbol V2_Capacitor:0805_10u -> V2_Capacitor:2012_10u
- D101: symbol V2_LED:0603_Orange -> V2_LED:1608_Orange
- R101: footprint V2_Resistor_SMD:R_0603 -> V2_Resistor_SMD:R_1608; symbol V2_Resistor:0603_100k -> V2_Resistor:1608_100k
- R102: footprint V2_Resistor_SMD:R_0603 -> V2_Resistor_SMD:R_1608; symbol V2_Resistor:0603_330R -> V2_Resistor:1608_330R
Changed lines of the file:
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@@
 	)
 	(symbol
-		(lib_id "V2_Capacitor:0603_0u1")
+		(lib_id "V2_Capacitor:1608_0u1")
 		(at 88.9 22.86 0)
 		(unit 1)
@@
 			)
 		)
-		(property "Footprint" "V2_Capacitor_SMD:C_0603"
+		(property "Footprint" "V2_Capacitor_SMD:C_1608"
 			(at 88.9 39.878 0)
 			(hide yes)
@@
 	)
 	(symbol
-		(lib_id "V2_LED:0603_Orange")
+		(lib_id "V2_LED:1608_Orange")
 		(at 132.08 55.88 0)
 		(mirror y)
@@
 	)
 	(symbol
-		(lib_id "V2_Capacitor:0805_10u")
+		(lib_id "V2_Capacitor:2012_10u")
 		(at 201.93 40.64 0)
 		(unit 1)
@@
 			)
 		)
-		(property "Footprint" "V2_Capacitor_SMD:C_0805"
+		(property "Footprint" "V2_Capacitor_SMD:C_2012"
 			(at 201.93 57.658 0)
 			(hide yes)
@@
 	)
 	(symbol
-		(lib_id "V2_Capacitor:0603_18p")
+		(lib_id "V2_Capacitor:1608_18p")
 		(at 26.67 45.72 0)
 		(unit 1)
@@
 			)
 		)
-		(property "Footprint" "V2_Capacitor_SMD:C_0603"
+		(property "Footprint" "V2_Capacitor_SMD:C_1608"
 			(at 26.67 62.738 0)
 			(hide yes)
@@
 	)
 	(symbol
-		(lib_id "V2_Capacitor:0805_10u")
+		(lib_id "V2_Capacitor:2012_10u")
 		(at 177.8 40.64 0)
 		(unit 1)
@@
 			)
 		)
-		(property "Footprint" "V2_Capacitor_SMD:C_0805"
+		(property "Footprint" "V2_Capacitor_SMD:C_2012"
 			(at 177.8 57.658 0)
 			(hide yes)
@@
 	)
 	(symbol
-		(lib_id "V2_Capacitor:0603_0u1")
+		(lib_id "V2_Capacitor:1608_0u1")
 		(at 119.38 22.86 0)
 		(unit 1)
@@
 			)
 		)
-		(property "Footprint" "V2_Capacitor_SMD:C_0603"
+		(property "Footprint" "V2_Capacitor_SMD:C_1608"
 			(at 119.38 39.878 0)
 			(hide yes)
@@
 	)
 	(symbol
-		(lib_id "V2_Resistor:0603_100k")
+		(lib_id "V2_Resistor:1608_100k")
 		(at 50.8 120.65 90)
 		(unit 1)
@@
 			)
 		)
-		(property "Footprint" "V2_Resistor_SMD:R_0603"
+		(property "Footprint" "V2_Resistor_SMD:R_1608"
 			(at 66.548 120.65 0)
 			(hide yes)
@@
 	)
 	(symbol
-		(lib_id "V2_Capacitor:0603_18p")
+		(lib_id "V2_Capacitor:1608_18p")
 		(at 21.59 45.72 0)
 		(unit 1)
@@
 			)
 		)
-		(property "Footprint" "V2_Capacitor_SMD:C_0603"
+		(property "Footprint" "V2_Capacitor_SMD:C_1608"
 			(at 21.59 62.738 0)
 			(hide yes)
@@
 	)
 	(symbol
-		(lib_id "V2_Resistor:0603_330R")
+		(lib_id "V2_Resistor:1608_330R")
 		(at 139.7 55.88 90)
 		(unit 1)
@@
 			)
 		)
-		(property "Footprint" "V2_Resistor_SMD:R_0603"
+		(property "Footprint" "V2_Resistor_SMD:R_1608"
 			(at 155.448 55.88 0)
 			(hide yes)
@@
 	)
 	(symbol
-		(lib_id "V2_Capacitor:0603_0u1")
+		(lib_id "V2_Capacitor:1608_0u1")
 		(at 99.06 22.86 0)
 		(unit 1)
@@
 			)
 		)
-		(property "Footprint" "V2_Capacitor_SMD:C_0603"
+		(property "Footprint" "V2_Capacitor_SMD:C_1608"
 			(at 99.06 39.878 0)
 			(hide yes)
@@
 	)
 	(symbol
-		(lib_id "V2_Capacitor:0603_0u1")
+		(lib_id "V2_Capacitor:1608_0u1")
 		(at 78.74 22.86 0)
 		(unit 1)
@@
 			)
 		)
-		(property "Footprint" "V2_Capacitor_SMD:C_0603"
+		(property "Footprint" "V2_Capacitor_SMD:C_1608"
 			(at 78.74 39.878 0)
 			(hide yes)
@@
 	)
 	(symbol
-		(lib_id "V2_Capacitor:0603_0u1")
+		(lib_id "V2_Capacitor:1608_0u1")
 		(at 109.22 22.86 0)
 		(unit 1)
@@
 			)
 		)
-		(property "Footprint" "V2_Capacitor_SMD:C_0603"
+		(property "Footprint" "V2_Capacitor_SMD:C_1608"
 			(at 109.22 39.878 0)
 			(hide yes)
@@
 	)
 	(symbol
-		(lib_id "V2_Capacitor:0603_10u")
+		(lib_id "V2_Capacitor:1608_10u")
 		(at 57.15 22.86 0)
 		(unit 1)
@@
 			)
 		)
-		(property "Footprint" "V2_Capacitor_SMD:C_0603"
+		(property "Footprint" "V2_Capacitor_SMD:C_1608"
 			(at 57.15 39.878 0)
 			(hide yes)
